Commit message: changes nov 28

File: rrbot_description/gazebo/rrbot.gazebo.xacro (robot description, xacro)
@@ -5,9 +5,9 @@
 -->
 <robot xmlns:xacro="http://ros.org/wiki/xacro">
-  <xacro:macro name="rrbot_gazebo" params="prefix">
+  <xacro:macro name="rrrbot_gazebo" params="prefix">
     <!-- ros_control plugin -->
     <gazebo>
       <plugin name="gazebo_ros2_control" filename="libgazebo_ros2_control.so">
-        <parameters>$(find rrbot_gazebo)/config/gazebo_controllers.yaml</parameters>
+        <parameters>$(find rrrbot_gazebo)/config/gazebo_controllers.yaml</parameters>
       </plugin>
     </gazebo>

File: rrbot_description/ros2_control/rrbot.ros2_control.xacro (robot description, xacro)
@@ -1,5 +1,5 @@
 <?xml version="1.0"?>
 <robot xmlns:xacro="http://www.ros.org/wiki/xacro">
-  <xacro:macro name="rrbot_ros2_control" params="name prefix">
+  <xacro:macro name="rrrbot_ros2_control" params="name prefix">
     <ros2_control name="${name}" type="system">
       <!-- <hardware>

File: rrbot_description/urdf/rrbot.urdf.xacro (robot description, xacro)
@@ -22,6 +22,6 @@
     <origin xyz="0 0 0" rpy="0 0 0" />
   </xacro:rrbot>
-  <xacro:rrbot_gazebo prefix="$(arg prefix)" />
-  <xacro:rrbot_ros2_control
+  <xacro:rrrbot_gazebo prefix="$(arg prefix)" />
+  <xacro:rrrbot_ros2_control
     name="RRBot" prefix="$(arg prefix)" />
 </robot>
