Commit message: working controller 30 nov

File: rrbot_description/urdf/rrbot_description.urdf.xacro (robot description, xacro)
@@ -105,8 +105,8 @@
         <parent link="${prefix}link2"/>
         <child link="${prefix}link3"/>
-        <limit effort="1000.0" lower="-0.38" upper="0.5" velocity="0.5"/>
+        <limit effort="1000.0" lower="-0.38" upper="0" velocity="0.5"/>
         <origin xyz="0 ${width} ${height3 - axel_offset*2}" rpy="0 0 0"/>
         <axis xyz="1 0 0"/>
-        <dynamics damping="0.7"/>
+        <dynamics damping="0.7" friction="11"/>
       </joint>
       <!-- Prismatic Link -->
